File: ESP32-DEVKIT-L/ESP32-DEVKIT-L.kicad_sch (KiCad schematic)
At the start: 132 parts, among them CON1 NA(NH1x20), J1 Conn_02x02_P4.20mm_Molex_Hori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, Q1 Q12MHz/20pF/30ppm/2P/HC-49SM(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, Q2 BC817-40(SOT23), Q3 BC817-40(SOT23), T1 DTC114YKA, U1 USB-C-16P-F(A40-00119-A52-12), U2 Converter_DCDC_RECOM_R-78HB-0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, U3 CH340T(SSOP20W), U4 LAN8710A-EZC(QFN32), U5 K7803-2000R3L, U6 TCA9548APWR, U7 ESP32-WROOM-32D-4MB

Commit message: 23.04.23
Connections:
- net GPI34\BUT1 renamed GPIO34\BUT1
- net GPI35 renamed GPIO35
- net GPI36 renamed GPIO36
- net GPI39 renamed GPIO39
Other:
- note added: "PHY_PWR/GPIO5:"
- note removed: "GPIO5\PHY_PWR:"
Changed lines of the file:
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@@
     (effects (font (size 0.9906 0.9906) italic) (justify left bottom))
   )
-  (text "MTDO/GPIO15:" (at 470.408 367.284 0)
+  (text "MTDO/GPIO15:" (at 470.408 367.538 0)
     (effects (font (size 1.4986 1.4986)) (justify left bottom))
   )
@@
     (effects (font (size 0.9906 0.9906) italic) (justify left bottom))
   )
-  (text "MTDI/GPIO12:" (at 471.678 352.044 0)
+  (text "MTDI/GPIO12:" (at 471.17 352.044 0)
     (effects (font (size 1.4986 1.4986)) (justify left bottom))
   )
@@
     (effects (font (size 1.0922 1.0922)) (justify left bottom))
   )
-  (text "GPIO4:" (at 479.298 363.474 0)
+  (text "GPIO4:" (at 479.298 363.728 0)
     (effects (font (size 1.4986 1.4986)) (justify left bottom))
   )
@@
     (effects (font (size 1.524 1.524)) (justify left bottom))
   )
-  (text "GPIO5\\PHY_PWR:" (at 479.298 371.094 0)
+  (text "PHY_PWR/GPIO5:" (at 467.614 371.348 0)
     (effects (font (size 1.4986 1.4986)) (justify left bottom))
   )
@@
     (effects (font (size 0.889 0.889)) (justify left bottom))
   )
-  (label "GPI34\\BUT1" (at 508.762 179.324 0) (fields_autoplaced)
+  (label "GPIO34\\BUT1" (at 508.762 179.324 0) (fields_autoplaced)
     (effects (font (size 0.9906 0.9906)) (justify left bottom))
   )
@@
     (effects (font (size 1.27 1.27)) (justify left bottom))
   )
-  (label "GPI35" (at 473.71 92.964 0) (fields_autoplaced)
+  (label "GPIO35" (at 473.71 92.964 0) (fields_autoplaced)
     (effects (font (size 1.27 1.27)) (justify left bottom))
   )
@@
     (effects (font (size 0.889 0.889)) (justify right bottom))
   )
-  (label "GPI36" (at 473.71 95.504 0) (fields_autoplaced)
+  (label "GPIO36" (at 473.71 95.504 0) (fields_autoplaced)
     (effects (font (size 1.27 1.27)) (justify left bottom))
   )
@@
     (effects (font (size 0.889 0.889)) (justify left bottom))
   )
-  (label "GPI34\\BUT1" (at 473.71 90.424 0) (fields_autoplaced)
+  (label "GPIO34\\BUT1" (at 473.71 90.424 0) (fields_autoplaced)
     (effects (font (size 1.2446 1.2446)) (justify left bottom))
   )
-  (label "GPI35" (at 396.24 121.92 0) (fields_autoplaced)
+  (label "GPIO35" (at 396.24 121.92 0) (fields_autoplaced)
     (effects (font (size 1.27 1.27)) (justify left bottom))
   )
@@
     (effects (font (size 1.27 1.27)) (justify left bottom))
   )
-  (label "GPI39" (at 473.71 98.044 0) (fields_autoplaced)
+  (label "GPIO39" (at 473.71 98.044 0) (fields_autoplaced)
     (effects (font (size 1.27 1.27)) (justify left bottom))
   )
@@
     (effects (font (size 1.27 1.27)) (justify left bottom))
   )
-  (label "GPI36" (at 396.24 124.46 0) (fields_autoplaced)
+  (label "GPIO36" (at 396.24 124.46 0) (fields_autoplaced)
     (effects (font (size 1.27 1.27)) (justify left bottom))
   )
@@
     (effects (font (size 0.9906 0.9906)) (justify left bottom))
   )
-  (label "GPI39" (at 396.24 127 0) (fields_autoplaced)
+  (label "GPIO39" (at 396.24 127 0) (fields_autoplaced)
     (effects (font (size 1.27 1.27)) (justify left bottom))
   )
@@
     (effects (font (size 1.27 1.27)) (justify left bottom))
   )
-  (label "GPI34\\BUT1" (at 396.24 119.38 0) (fields_autoplaced)
-    (effects (font (size 1.27 1.27)) (justify left bottom))
-  )
+  (label "GPIO34\\BUT1" (at 396.24 119.38 0) (fields_autoplaced)
+    (effects (font (size 1.27 1.27)) (justify left bottom))
+  )
