File: Rev0/Rev0.kicad_pcb (KiCad board)
At the start: 2 copper layers, 71.7 x 72.8 mm, 142 parts, among them CON1 NA(NH1x20), J1 Conn_02x02_P4.20mm_Molex_Hori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, Q1 Q12MHz/20pF/30ppm/2P/HC-49SM(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, Q2 BC817-40(SOT23), Q3 BC817-40(SOT23), T1 DTC114YKA, U1 USB-C-16P-F(A40-00119-A52-12), U2 Converter_DCDC_RECOM_R-78HB-0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, U3 CH340T(SSOP20W), U4 LAN8710A-EZC(QFN32), U5 K7803-2000R3L, U6 TCA9548APWR, U7 ESP32-WROOM-32D-4MB

Commit message: .
Other:
- board text added: "V+"
- board text removed: "+12V"
Changed lines of the file:
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@@
     (fp_arc (start 2.54762 -5.59816) (mid 2.405726 -5.656926) (end 2.34696 -5.79882)
       (stroke (width 0.127) (type solid)) (layer "F.Fab"))
-    (fp_arc (start 3.66522 -5.715) (mid 3.534891 -5.62876) (end 3.381484 -5.598961)
+    (fp_arc (start 3.66522 -5.715) (mid 3.534891 -5.628772) (end 3.381484 -5.598961)
       (stroke (width 0.127) (type solid)) (layer "F.Fab"))
     (fp_arc (start 8.6487 -6.2992) (mid 9.214456 -6.064856) (end 9.4488 -5.4991)
@@
     (fp_arc (start 2.159 1.27) (mid 2.069197 1.232803) (end 2.032 1.143)
       (stroke (width 0.254) (type solid)) (layer "B.SilkS"))
-    (fp_arc (start 2.224065 2.284155) (mid 2.619863 2.433425) (end 2.921 2.7305)
+    (fp_arc (start 2.224065 2.284155) (mid 2.619862 2.433426) (end 2.921 2.7305)
       (stroke (width 0.254) (type solid)) (layer "B.SilkS"))
-    (fp_arc (start 2.224929 1.013456) (mid 2.269136 1.033818) (end 2.286 1.0795)
+    (fp_arc (start 2.224929 1.013456) (mid 2.269175 1.033812) (end 2.286 1.0795)
       (stroke (width 0.254) (type solid)) (layer "B.SilkS"))
     (fp_arc (start 2.286 1.2065) (mid 2.267401 1.251401) (end 2.2225 1.27)
@@
     (fp_arc (start 0.508 2.413) (mid -0.569631 1.966631) (end -1.016 0.889)
       (stroke (width 0.254) (type solid)) (layer "B.SilkS"))
-    (fp_arc (start 8.229048 7.764478) (mid 9.052754 7.423877) (end 9.9441 7.42442)
+    (fp_arc (start 8.229048 7.764478) (mid 9.052754 7.423879) (end 9.9441 7.42442)
       (stroke (width 0.254) (type solid)) (layer "B.SilkS"))
     (fp_arc (start 8.234536 6.260553) (mid 9.129375 4.989852) (end 10.21588 3.87858)
@@
     (fp_arc (start 9.042459 6.381222) (mid 10.012997 5.890291) (end 11.06932 5.63118)
       (stroke (width 0.254) (type solid)) (layer "B.SilkS"))
-    (fp_arc (start 10.153621 6.316813) (mid 10.819746 6.177307) (end 11.49604 6.10108)
+    (fp_arc (start 10.153621 6.316813) (mid 10.819745 6.177303) (end 11.49604 6.10108)
       (stroke (width 0.254) (type solid)) (layer "B.SilkS"))
     (fp_arc (start 10.255067 3.840987) (mid 11.121885 3.322842) (end 12.12088 3.175)
@@
     (fp_arc (start 12.319 -0.635) (mid 13.396631 -0.188631) (end 13.843 0.889)
       (stroke (width 0.254) (type solid)) (layer "B.SilkS"))
-    (fp_arc (start 12.6365 3.172934) (mid 12.92792 3.230905) (end 13.17498 3.39598)
+    (fp_arc (start 12.6365 3.172934) (mid 12.927926 3.230899) (end 13.17498 3.39598)
       (stroke (width 0.254) (type solid)) (layer "B.SilkS"))
     (fp_arc (start 13.27787 5.527066) (mid 12.666712 5.829464) (end 12.0142 6.02742)
       (stroke (width 0.254) (type solid)) (layer "B.SilkS"))
-    (fp_arc (start 13.718022 1.77772) (mid 14.092522 2.33979) (end 14.224 3.00228)
+    (fp_arc (start 13.718022 1.77772) (mid 14.092534 2.33979) (end 14.224 3.00228)
       (stroke (width 0.254) (type solid)) (layer "B.SilkS"))
-    (fp_arc (start 13.776451 2.089441) (mid 14.108184 2.587709) (end 14.224 3.175)
+    (fp_arc (start 13.776451 2.089441) (mid 14.108196 2.587709) (end 14.224 3.175)
       (stroke (width 0.254) (type solid)) (layer "B.SilkS"))
     (fp_arc (start 13.843 0.889) (mid 13.396631 1.966631) (end 12.319 2.413)
       (stroke (width 0.254) (type solid)) (layer "B.SilkS"))
-    (fp_arc (start 13.933527 4.300844) (mid 12.739662 5.103149) (end 11.3792 5.57022)
+    (fp_arc (start 13.933527 4.300844) (mid 12.739664 5.103156) (end 11.3792 5.57022)
       (stroke (width 0.254) (type solid)) (layer "B.SilkS"))
     (fp_arc (start 13.94714 3.45186) (mid 13.587204 3.599468) (end 13.22832 3.44932)
       (stroke (width 0.254) (type solid)) (layer "B.SilkS"))
-    (fp_arc (start 13.955743 2.395289) (mid 14.154815 2.694956) (end 14.224 3.048)
+    (fp_arc (start 13.955743 2.395289) (mid 14.154803 2.694956) (end 14.224 3.048)
       (stroke (width 0.254) (type solid)) (layer "B.SilkS"))
     (fp_arc (start 14.143264 6.107415) (mid 13.349685 7.17762) (end 12.09294 7.62)
@@
     (fp_arc (start 14.328866 2.561046) (mid 14.49285 2.451478) (end 14.68628 2.413)
       (stroke (width 0.254) (type solid)) (layer "B.SilkS"))
-    (fp_arc (start 14.344359 4.449235) (mid 13.859873 5.026773) (end 13.28928 5.51942)
+    (fp_arc (start 14.344359 4.449235) (mid 13.859872 5.026772) (end 13.28928 5.51942)
       (stroke (width 0.254) (type solid)) (layer "B.SilkS"))
-    (fp_arc (start 14.35024 4.826757) (mid 14.339076 5.167151) (end 14.29004 5.50418)
+    (fp_arc (start 14.35024 4.826757) (mid 14.339075 5.167151) (end 14.29004 5.50418)
       (stroke (width 0.254) (type solid)) (layer "B.SilkS"))
-    (fp_arc (start 14.68628 2.411388) (mid 14.844363 2.442831) (end 14.97838 2.53238)
+    (fp_arc (start 14.68628 2.411388) (mid 14.844369 2.442825) (end 14.97838 2.53238)
       (stroke (width 0.254) (type solid)) (layer "B.SilkS"))
     (fp_arc (start 14.730126 3.530099) (mid 14.751792 3.304011) (end 14.81582 3.0861)
       (stroke (width 0.254) (type solid)) (layer "B.SilkS"))
-    (fp_arc (start 14.859445 3.404629) (mid 14.925626 3.074154) (end 15.113 2.794)
+    (fp_arc (start 14.859445 3.404629) (mid 14.92562 3.074148) (end 15.113 2.794)
       (stroke (width 0.254) (type solid)) (layer "B.SilkS"))
     (fp_arc (start 14.932206 4.285679) (mid 14.782902 3.921185) (end 14.732 3.5306)
       (stroke (width 0.254) (type solid)) (layer "B.SilkS"))
-    (fp_arc (start 15.111212 2.665208) (mid 15.275779 2.698133) (end 15.41526 2.79146)
+    (fp_arc (start 15.111212 2.665208) (mid 15.275768 2.698145) (end 15.41526 2.79146)
       (stroke (width 0.254) (type solid)) (layer "B.SilkS"))
-    (fp_arc (start 15.38866 2.763954) (mid 15.702814 3.271585) (end 15.7988 3.8608)
+    (fp_arc (start 15.38866 2.763954) (mid 15.702828 3.271585) (end 15.7988 3.8608)
       (stroke (width 0.254) (type solid)) (layer "B.SilkS"))
     (fp_arc (start 15.67766 2.671387) (mid 16.007869 3.019303) (end 16.1798 3.4671)
       (stroke (width 0.254) (type solid)) (layer "B.SilkS"))
-    (fp_arc (start 15.708 5.025489) (mid 15.294548 4.762303) (end 14.986 4.3815)
+    (fp_arc (start 15.708 5.025489) (mid 15.294541 4.762306) (end 14.986 4.3815)
       (stroke (width 0.254) (type solid)) (layer "B.SilkS"))
-    (fp_arc (start 16.026073 2.665697) (mid 16.126536 2.671678) (end 16.22552 2.68986)
+    (fp_arc (start 16.026073 2.665697) (mid 16.126535 2.67168) (end 16.22552 2.68986)
       (stroke (width 0.254) (type solid)) (layer "B.SilkS"))
     (fp_arc (start 16.227503 2.690547) (mid 16.535892 2.788064) (end 16.80718 2.96418)
@@
     (fp_arc (start 16.559205 4.805934) (mid 16.306617 4.337511) (end 16.2052 3.81508)
       (stroke (width 0.254) (type solid)) (layer "B.SilkS"))
-    (fp_arc (start 16.831054 2.986026) (mid 17.063406 3.333768) (end 17.145 3.74396)
+    (fp_arc (start 16.831054 2.986026) (mid 17.063417 3.333768) (end 17.145 3.74396)
       (stroke (width 0.254) (type solid)) (layer "B.SilkS"))
     (fp_arc (start 17.009851 5.046864) (mid 16.968283 4.574521) (end 17.07388 4.11226)
       (stroke (width 0.254) (type solid)) (layer "B.SilkS"))
-    (fp_arc (start 17.144717 3.743513) (mid 17.126889 3.931265) (end 17.07388 4.11226)
+    (fp_arc (start 17.144717 3.743513) (mid 17.126897 3.931268) (end 17.07388 4.11226)
       (stroke (width 0.254) (type solid)) (layer "B.SilkS"))
   )
@@
     (effects (font (size 3.048 3.048) (thickness 0.635)) (justify left mirror))
   )
-  (gr_text "+12V" (at 118.32 90.915 90) (layer "B.SilkS")
+  (gr_text "GND" (at 129.86 90.915 90) (layer "B.SilkS")
+    (effects (font (size 1.5 1.5) (thickness 0.3)) (justify mirror))
+  )
+  (gr_text "V+" (at 118.32 90.915 90) (layer "B.SilkS")
     (effects (font (size 1.5 1.5) (thickness 0.3)) (justify mirror))
   )
@@
     (effects (font (size 0.762 0.762) (thickness 0.1905)))
   )
-  (gr_text "+12V" (at 118.32 91.125 90) (layer "F.SilkS")
+  (gr_text "V+" (at 121.34 96.095 90) (layer "F.SilkS")
+    (effects (font (size 1.5 1.5) (thickness 0.3)))
+  )
+  (gr_text "GND" (at 126.84 96.885 90) (layer "F.SilkS")
     (effects (font (size 1.5 1.5) (thickness 0.3)))
   )
@@
   (segment (start 109.215 120.909) (end 108.331 121.793) (width 0.254) (layer "F.Cu") (net 18))
   (segment (start 109.474 120.909) (end 109.215 120.909) (width 0.254) (layer "F.Cu") (net 18))
+  (segment (start 105.3465 120.736) (end 104.719 120.736) (width 0.3048) (layer "F.Cu") (net 19))
   (segment (start 105.3465 120.736) (end 107.274 120.736) (width 0.254) (layer "F.Cu") (net 19))
-  (segment (start 104.4067 120.736) (end 104.267 120.8757) (width 0.3048) (layer "F.Cu") (net 19))
+  (segment (start 104.38 122.95) (end 102.8065 124.5235) (width 0.3048) (layer "F.Cu") (net 19))
   (segment (start 107.274 120.736) (end 107.442 120.904) (width 0.254) (layer "F.Cu") (net 19))
-  (segment (start 105.3465 120.736) (end 104.4067 120.736) (width 0.3048) (layer "F.Cu") (net 19))
-  (segment (start 104.267 123.063) (end 102.8065 124.5235) (width 0.3048) (layer "F.Cu") (net 19))
-  (segment (start 104.267 120.8757) (end 104.267 123.063) (width 0.3048) (layer "F.Cu") (net 19))
   (segment (start 102.8065 124.5235) (end 102.616 124.5235) (width 0.3048) (layer "F.Cu") (net 19))
+  (segment (start 104.38 121.075) (end 104.38 122.95) (width 0.3048) (layer "F.Cu") (net 19))
+  (segment (start 104.719 120.736) (end 104.38 121.075) (width 0.3048) (layer "F.Cu") (net 19))
   (segment (start 80.38348 98.1903) (end 80.38348 99.34966) (width 0.2032) (layer "F.Cu") (net 20))
   (segment (start 81.802865 116.3523) (end 81.826665 116.3761) (width 0.2032) (layer "F.Cu") (net 20))

Commit message: .
Parts:
- removed G*** (x2): LOGO, Hasat.io:Hasatio_logo_mini
- removed G***: LOGO, Hasat.io:Hasatio
- removed G***: LOGO, Hasat.io:esp-devkit-l
- removed LED: Closed, OLIMEX_Jumpers-FP:SJ
- removed RESET: Opened, OLIMEX_Jumpers-FP:SJ
- added ?: , , F.Cu at (118.9, 124.1)
- added FID1: Fiducial, OLIMEX_Other-FP:Fiducial1x3, F.Cu at (77.5, 124.1)
- added FID3: Fiducial, OLIMEX_Other-FP:Fiducial1x3, F.Cu at (117.4, 75.9)
- added LED_E1: Closed, OLIMEX_Jumpers-FP:SJ, B.Cu at (116.1, 86.3)
- added PHY_RST1: Opened, OLIMEX_Jumpers-FP:SJ, B.Cu at (105.7, 100.5)
- added R3: 0R(Board_Mounted), Resistors:0603, F.Cu at (104.8, 91.7)
- C23: value 100nF/50V/20%/Y5V/C0603 -> 100nF/6.3V/20%/X5R/C0603
- L1: value FB0805/600R/2A -> NA(FB0805/600R/2A)
- R25: renamed from R26; value 4.7k/R0603 -> 2.2k/R0603
- R27: renamed from R28; value 4.7k/R0603 -> 2.2k/R0603
- U1: renamed from U2; value Converter_DCDC_RECOM_R-78HB-0.5L_THT -> K7805-2000R3L; footprint Converter_DCDC:Converter_DCDC_RECOM_R-78HB-0.5L_THT -> K7812-2000R3L:K78122000R3L
- U4: renamed from U5; footprint Converter_DCDC:Converter_DCDC_RECOM_R-78HB-0.5L_THT -> K7812-2000R3L:K78122000R3L
- moved Sign_Pb-Free 49.2 mm to (139.3, 130.9)
- moved Sign_RoHS 33.8 mm to (139.4, 138.4)
- moved Sign-Antistatic 20.9 mm to (128.2, 81.2)
- moved Sign-RecyclBin 12.5 mm to (127.0, 88.0)
- moved R15 5.26 mm to (94.9, 118.7), turned to 180 degrees
- moved C15 2.55 mm to (104.5, 94.2), turned to 0 degrees
- moved C7 2.40 mm to (94.9, 121.2), turned to 180 degrees
- moved J1 1.86 mm to (126.6, 90.8)
- moved REF** 1.86 mm to (126.6, 90.8)
- moved C1 0.76 mm to (135.2, 74.7)
- moved REF** 0.59 mm to (127.5, 108.3)
- moved U1 0.54 mm to (121.2, 108.4), turned to 0 degrees
- moved C29 0.13 mm to (79.8, 132.2)
- moved C31 0.13 mm to (119.7, 132.2)
- moved C27 0.13 mm to (111.8, 132.2)
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- renumbered C9 to C10, C27 to C26, C29 to C27, C31 to C28, C26 to C29, C28 to C30, C30 to C31, C10 to C6, C6 to C7, C7 to C8, C8 to C9, I²C0 to J2, I²C2 to J3, I²C4 to J4, I²C6 to J5, I²C1 to J6, I²C3 to J7, I²C5 to J8, I²C7 to J9, R11 to R10, R12 to R11, R13 to R12, R14 to R13, R15 to R14, R16 to R15, R17 to R16, R18 to R17, R19 to R18, R20 to R19, R21 to R20, R22 to R21, R23 to R22, R24 to R23, R25 to R24, R27 to R26, R37 to R28, R31 to R30, R43 to R31, R45 to R32, R38 to R33, R41 to R34, R42 to R35, R33 to R36, R35 to R37, R47 to R38, R49 to R39, R5 to R4, R39 to R40, R40 to R41, R30 to R42, R32 to R43, R46 to R45, R50 to R46, R34 to R47, R36 to R48, R48 to R49, R6 to R5, R51 to R50, R52 to R51, R53 to R52, R3 to R53, R4 to R54, R7 to R6, R8 to R7, R9 to R8, R10 to R9, U3 to U2, U4 to U3, U6 to U5, U7 to U6, U1 to U7
Connections:
- net /SC0 renamed Net-(J2-Pad4)
- net /SC1 renamed Net-(J6-Pad4)
- net /SC2 renamed Net-(J3-Pad4)
- net /SC3 renamed Net-(J7-Pad4)
- net /SC4 renamed Net-(J4-Pad4)
- net /SC5 renamed Net-(J8-Pad4)
- net /SC6 renamed Net-(J5-Pad4)
- net /SC7 renamed Net-(J9-Pad4)
- net /SD0 renamed Net-(J2-Pad3)
- net /SD1 renamed Net-(J6-Pad3)
- net /SD2 renamed Net-(J3-Pad3)
- net /SD3 renamed Net-(J7-Pad3)
- net /SD4 renamed Net-(J4-Pad3)
- net /SD5 renamed Net-(J8-Pad3)
- net /SD6 renamed Net-(J5-Pad3)
- net /SD7 renamed Net-(J9-Pad3)
- C30 pad 1: +3V3 -> GND
- C30 pad 2: GND -> +3V3
Routing:
- net GND: track 482.3 -> 625.3 mm, vias 328 -> 426
- net +3V3: track 639.4 -> 570.9 mm, vias 9 -> 12
- net /+5V_USB: track 128.1 -> 87.1 mm
- net +3.3VLAN: track 78.7 -> 50.4 mm
- net /GPIO2\HS2_DATA0: track 71.3 -> 56.5 mm
- net Net-(C1-Pad1): track 56.0 -> 42.8 mm
- net +5V: track 66.0 -> 57.7 mm
- net Net-(Q2-Pad2): track 22.9 -> 15.1 mm
- net /ESP_EN: track 98.0 -> 90.8 mm, vias 4 -> 3
- net /GPIO5\PHY_PWR: track 69.2 -> 75.0 mm
- net /GPIO23\MDC(RMII): track 40.5 -> 45.8 mm
- net /GPIO4\HS2_DATA1: track 64.2 -> 59.0 mm
- net /VDD1A-2A: track 110.1 -> 114.7 mm
- net Net-(J4-Pad3): track 17.2 -> 13.1 mm
- net /GPIO22\EMAC_TXD1(RMII): track 35.7 -> 39.5 mm
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Other:
- rule pad_to_mask_clearance: 0 -> 0.2
- board text added: "(C) 2022"
- board text added: "ESP32-GATEWAY"
- board text added: "Rev.0"
- board text removed: "(C) 2023"
- board text removed: "ESP32-DEVKIT-L"
- board text removed: "Rev.1"
- board text removed: "V+"

Commit message: .
Parts:
- C23: value 100nF/6.3V/20%/X5R/C0603 -> 100nF/6.3V/20%/X5R/C0805; footprint Capacitors:0603 -> Capacitors:0805
- C25, C26, C27, C28, C29, C30, C31, C32: value 1uF/6.3V/20%/X5R/C0603 -> 1uF/6.3V/20%/X5R/C0805; footprint Capacitors:0603 -> Capacitors:0805
- moved J9 55.6 mm to (81.6, 136.4)
- moved C28 55.6 mm to (71.9, 132.2)
- moved J5 55.6 mm to (73.7, 136.4)
- moved R32 55.6 mm to (74.2, 131.4)
- moved R39 55.6 mm to (75.7, 131.4)
- moved R46 55.6 mm to (83.5, 131.4)
- moved C32 55.6 mm to (79.8, 132.2)
- moved R45 55.6 mm to (82.1, 131.4)
- moved C26 24.3 mm to (111.8, 132.2)
- moved J7 24.2 mm to (121.5, 136.4)
- moved R43 24.2 mm to (122.0, 131.4)
- moved C30 24.2 mm to (119.7, 132.2)
- moved R48 24.2 mm to (123.4, 131.4)
- moved J3 24.2 mm to (113.6, 136.4)
- moved R30 24.2 mm to (114.1, 131.4)
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Routing:
- net Net-(J2-Pad3): track 37.2 -> 19.7 mm
- net Net-(J8-Pad4): track 23.9 -> 40.5 mm
- net Net-(J6-Pad3): track 29.1 -> 13.2 mm
- net Net-(J8-Pad3): track 21.3 -> 36.5 mm
- net Net-(J2-Pad4): track 34.8 -> 19.7 mm
- net Net-(J4-Pad4): track 16.0 -> 31.0 mm
- net Net-(J6-Pad4): track 26.8 -> 13.7 mm
- net Net-(J9-Pad4): track 39.9 -> 27.0 mm
- net Net-(J4-Pad3): track 13.1 -> 25.8 mm
- net +3V3: track 570.9 -> 582.5 mm
- net Net-(J5-Pad3): track 28.9 -> 38.1 mm
- net Net-(J7-Pad4): track 11.3 -> 20.5 mm
- net Net-(J9-Pad3): track 36.8 -> 28.0 mm
- net Net-(J3-Pad3): track 21.0 -> 13.7 mm
- net Net-(J7-Pad3): track 13.1 -> 20.2 mm
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