File: Rev0/Rev0.kicad_sch (KiCad schematic)
At the start: 132 parts, among them CON1 NA(NH1x20), J1 Conn_02x02_P4.20mm_Molex_Hori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, Q1 Q12MHz/20pF/30ppm/2P/HC-49SM(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, Q2 BC817-40(SOT23), Q3 BC817-40(SOT23), T1 DTC114YKA, U1 USB-C-16P-F(A40-00119-A52-12), U2 Converter_DCDC_RECOM_R-78HB-0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, U3 CH340T(SSOP20W), U4 LAN8710A-EZC(QFN32), U5 K7803-2000R3L, U6 TCA9548APWR, U7 ESP32-WROOM-32D-4MB

Commit message: .
Parts:
- U2: value Converter_DCDC_RECOM_R-78HB-0.5L_THT -> K7805-2000R3L

Commit message: .
Parts:
- removed LED: Closed, OLIMEX_Jumpers-FP:SJ, symbol ESP32-GATEWAY_Rev_G:SJ
- removed R14: 2.2k/R0603, Resistors:0603, symbol ESP32-GATEWAY_Rev_G:R
- removed U2: K7805-2000R3L, Converter_DCDC:Converter_DCDC_RECOM_R-78HB-0.5L_THT, symbol Regulator_Switching:R-78B5.0-2.0
- removed U5: K7803-2000R3L, Converter_DCDC:Converter_DCDC_RECOM_R-78HB-0.5L_THT, symbol Regulator_Switching:R-78B3.3-2.0
- added LED_E1: Closed, OLIMEX_Jumpers-FP:SJ, symbol ESP32-GATEWAY_Rev_G:SJ
- added R12: 1M/R0603, Resistors:0603, symbol ESP32-GATEWAY_Rev_G:R
- added R3: 0R(Board_Mounted), Resistors:0603, symbol ESP32-GATEWAY_Rev_G:R
- added U1: K7805-2000R3L, K7812-2000R3L:K78122000R3L, symbol Regulator_Switching:R-78B5.0-2.0
- added U4: K7803-2000R3L, K7812-2000R3L:K78122000R3L, symbol Regulator_Switching:R-78B3.3-2.0
- added USB-UART1: MISB-SWMM-5B-LF(USB_MICRO), OLIMEX_Connectors-FP:USB-MICRO_MISB-SWMM-5B_LF, symbol ESP32-GATEWAY_Rev_G:USB-MINI
- C23: value 100nF/50V/20%/Y5V/C0603 -> 100nF/6.3V/20%/X5R/C0603
- L1: value FB0805/600R/2A -> NA(FB0805/600R/2A)
- R13: value 1M/R0603 -> 2.2k/R0603
- renumbered C9 to C10, C27 to C26, C29 to C27, C31 to C28, C26 to C29, C28 to C30, C30 to C31, C10 to C6, C6 to C7, C7 to C8, C8 to C9, I²C0 to J2, I²C2 to J3, I²C4 to J4, I²C6 to J5, I²C1 to J6, I²C3 to J7, I²C5 to J8, I²C7 to J9, RESET to PHY_RST1, R11 to R10, R12 to R11, R15 to R14, R16 to R15, R17 to R16, R18 to R17, R19 to R18, R20 to R19, R21 to R20, R22 to R21, R23 to R22, R24 to R23, R25 to R24, R26 to R25, R27 to R26, R28 to R27, R37 to R28, R31 to R30, R43 to R31, R45 to R32, R38 to R33, R41 to R34, R42 to R35, R33 to R36, R35 to R37, R47 to R38, R49 to R39, R5 to R4, R39 to R40, R40 to R41, R30 to R42, R32 to R43, R46 to R45, R50 to R46, R34 to R47, R36 to R48, R48 to R49, R6 to R5, R51 to R50, R52 to R51, R53 to R52, R3 to R53, R4 to R54, R7 to R6, R8 to R7, R9 to R8, R10 to R9, U3 to U2, U4 to U3, U6 to U5, U7 to U6, U1 to U7
Connections:
- net +3V3: now also C30.2, U4.3 (OUT); no longer C30.1
- net +5V: now also LED_E1.1, LED_E1.2, U4.1 (IN)
- net +5V_EXT: now also R12.1, U1.3 (OUT); no longer R13.1
- net +5V_USB: now also USB-UART1.1 (VBUS)
- net GND: now also C30.1, R12.2, U1.2 (GND), U4.2 (GND), USB-UART1.0, USB-UART1.5 (GND); no longer C30.2
- net VDD1A-2A: now also R3.1, R3.2
- net at U2.6 (UD+), U7.A6 (DP1), U7.B6 (DP2): now also USB-UART1.3 (D+)
- net at U2.7 (UD-), U7.A7 (DN1), U7.B7 (DN2): now also USB-UART1.2 (D-)
- net at PWRLED1.1 (K): now also R13.1
- net at C1.1, J1.3 (Pin_3), J1.4 (Pin_4): now also U1.1 (IN)
- net GPIO34\BUT1 renamed GPI34\BUT1
- net GPIO35 renamed GPI35
- net GPIO36 renamed GPI36
- net GPIO39 renamed GPI39
- net SC0: no longer names the net of J2.4 (Pin_4), R36.2, U5.5 (SC0)
- net SC1: no longer names the net of J6.4 (Pin_4), R47.2, U5.7 (SC1)
- net SC2: no longer names the net of J3.4 (Pin_4), R37.2, U5.9 (SC2)
- net SC3: no longer names the net of J7.4 (Pin_4), R48.2, U5.11 (SC3)
- net SC4: no longer names the net of J4.4 (Pin_4), R38.2, U5.14 (SC4)
- net SC5: no longer names the net of J8.4 (Pin_4), R49.2, U5.16 (SC5)
- net SC6: no longer names the net of J5.4 (Pin_4), R39.2, U5.18 (SC6)
- net SC7: no longer names the net of J9.4 (Pin_4), R46.2, U5.20 (SC7)
- net SD0: no longer names the net of J2.3 (Pin_3), R29.2, U5.4 (SD0)
- net SD1: no longer names the net of J6.3 (Pin_3), R42.2, U5.6 (SD1)
- net SD2: no longer names the net of J3.3 (Pin_3), R30.2, U5.8 (SD2)
- net SD3: no longer names the net of J7.3 (Pin_3), R43.2, U5.10 (SD3)
- net SD4: no longer names the net of J4.3 (Pin_3), R31.2, U5.13 (SD4)
- net SD5: no longer names the net of J8.3 (Pin_3), R44.2, U5.15 (SD5)
- net SD6: no longer names the net of J5.3 (Pin_3), R32.2, U5.17 (SD6)
- net SD7: no longer names the net of J9.3 (Pin_3), R45.2, U5.19 (SD7)
- no-connect marks 17 -> 18
Other:
- note added: "GPIO5\PHY_PWR:"
- note removed: "PHY_PWR/GPIO5:"
- company: HASATIO -> OLIMEX LTD.
- title: ESP32-DEVKIT-L -> ESP32-GATEWAY
- moved on the sheet: BUT1, C12, C13, C14, C15, C16, C17, C18, C2, C20, C23, C25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

Commit message: .
Other:
- company: OLIMEX LTD. -> HASATIO
- title: ESP32-GATEWAY -> ESP32-DEVKIT-L
