File: Rev1/Rev1.kicad_sch (KiCad schematic)
At the start: 132 parts, among them CON1 NA(NH1x20), J1 Conn_02x02_P4.20mm_Molex_Hori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, Q1 Q12MHz/20pF/30ppm/2P/HC-49SM(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, Q2 BC817-40(SOT23), Q3 BC817-40(SOT23), T1 DTC114YKA, U1 USB-C-16P-F(A40-00119-A52-12), U2 K7805-2000R3L, U3 CH340T(SSOP20W), U4 LAN8710A-EZC(QFN32), U5 K7803-2000R3L, U6 TCA9548APWR, U7 ESP32-WROOM-32D-4MB

Commit message: .
Parts:
- renumbered LED2 to LED, RESET1 to RESET
Connections:
- net GPIO16: now also R26.2, U6.23 (SDA)
- net GPIO33 renamed GPIO33\LED
- net GPIO33\LED: now also LED1.2 (A); no longer R26.2, U6.23 (SDA)
- net GPIO35\LED renamed GPIO35
- net GPIO35: no longer LED1.2 (A)
