File: Rev2/Rev2.kicad_pcb (KiCad board)
At the start: 2 copper layers, 71.7 x 72.8 mm, 142 parts, among them CON1 NA(NH1x20), J1 Conn_02x02_P4.20mm_Molex_Hori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, Q1 Q12MHz/20pF/30ppm/2P/HC-49SM(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, Q2 BC817-40(SOT23), Q3 BC817-40(SOT23), T1 DTC114YKA, U1 USB-C-16P-F(A40-00119-A52-12), U2 K7805-2000R3L, U3 CH340T(SSOP20W), U4 LAN8710A-EZC(QFN32), U5 K7803-2000R3L, U6 TCA9548APWR, U7 ESP32-WROOM-32D-4MB

Commit message: .
Parts:
- moved GND1 5.07 mm to (113.8, 77.9)
- moved R4 1.35 mm to (128.9, 77.5), turned to 90 degrees
- moved R16 1.34 mm to (91.1, 122.0), turned to 0 degrees
- moved C6 1.22 mm to (95.7, 122.0), turned to 180 degrees
- moved D5 1.18 mm to (86.2, 98.4)
- moved R3 1.11 mm to (120.3, 77.5), turned to 90 degrees
- moved L1 0.69 mm to (85.4, 102.2)
- moved R23 0.21 mm to (86.5, 104.9)
- moved R20 0.17 mm to (82.3, 100.4)
- moved R24 0.13 mm to (86.5, 106.3)
Connections:
- net /GPIO32 renamed /GPIO32/SCL
- net /GPIO33 renamed /GPIO33/SDA
Routing:
- net +3V3: track 721.5 -> 708.7 mm
- net GND: track 482.3 -> 472.2 mm, vias 328 -> 329
- net +5V_EXT: track 65.6 -> 71.7 mm
- net /GPIO2\HS2_DATA0: track 71.3 -> 65.6 mm
- net /D_Com: track 34.4 -> 31.3 mm
- net Net-(Q2-E): track 22.9 -> 20.6 mm
- net /GPIO0: track 12.4 -> 10.3 mm
- net Net-(U1-CC1): track 11.7 -> 10.3 mm
- net +3.3VLAN: track 78.7 -> 80.0 mm
- net /GPIO16: track 54.1 -> 53.3 mm
Other:
- board text added: "Rev.2"
- board text removed: "Rev.1"

Commit message: .
Routing:
- net +3V3: track 708.7 -> 850.7 mm
- net GND: track 472.2 -> 475.1 mm, vias 329 -> 321
- net +5V_EXT: track 71.7 -> 70.6 mm

Commit message: .
Parts:
- moved C6 1.07 mm to (96.6, 121.5), turned to 90 degrees
- moved R15 0.79 mm to (95.7, 117.0)
Routing:
- net Net-(Q2-B): track 2.02 -> 2.85 mm
